File: Bread power Supply.kicad_sch (KiCad schematic)
At the start: 17 parts, among them J1 Conn_01x02_Pin, J2 Conn_01x02_Pin, J3 Conn_01x03_Pin, J4 Conn_01x03_Pin, J5 Screw_Terminal_01x02, J6 Barrel_Jack_Switch, J7 Screw_Terminal_01x02, U1 LM7805_TO220, U2 LM317_TO-220

Commit message: update
Other:
- title: Breadboard Power Supply -> ${project_name}
Changed lines of the file:
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@@
 	(paper "A4")
 	(title_block
-		(title "Breadboard Power Supply")
+		(title "${project_name}")
 		(date "2025-12-19")
 		(rev "Version 1")
